Commit message: update

File: install/yzbot_description/share/yzbot_description/urdf/yzbot_base.urdf (robot description, URDF)
Before this commit: robot yzbot, 6 links, 5 joints
Links:
- removed link caster_link
- added link base_footprint
- added link caster_back_link, mass 0.02; collision sphere radius=0.035; visual sphere radius=0.035
- added link caster_front_link, mass 0.02; collision sphere radius=0.035; visual sphere radius=0.035
- added link pic_link; visual box size=0.02 0.02 0.05
- link base_link: mass None -> 0.2; geometry collision box size=0.4 0.39 0.5; visual box size=0.4 0.39 0.5
- link imu_link: mass None -> 0.1; geometry collision box size=0.02 0.02 0.02; visual box size=0.02 0.02 0.02
- link laser_link: mass None -> 0.1; geometry collision cylinder length=0.02 radius=0.02; visual cylinder length=0.02 radius=0.02
- link left_wheel_link: mass None -> 0.2; geometry collision cylinder length=0.05 radius=0.07; visual cylinder length=0.05 radius=0.07
- link right_wheel_link: mass None -> 0.2; geometry collision cylinder length=0.05 radius=0.07; visual cylinder length=0.05 radius=0.07
Joints:
- removed joint caster_joint
- added joint base_joint: type fixed, parent base_footprint, child base_link, origin xyz=0.0 0.0 0.25 rpy=0 0 0
- added joint caster_back_joint: type fixed, parent base_link, child caster_back_link, origin xyz=-0.18 0.0 -0.285, axis 0 1 0
- added joint caster_front_joint: type fixed, parent base_link, child caster_front_link, origin xyz=0.18 0.0 -0.285, axis 0 1 0
- added joint joint_pic: type fixed, parent base_link, child pic_link, origin xyz=0.2 0.0 0.0 rpy=0 0 0
- joint laser_joint: origin xyz=0 0 0.075 -> xyz=0.0 0.0 0.265
- joint left_wheel_joint: origin xyz=-0.02 0.10 -0.06 -> xyz=0 0.2 -0.25
- joint right_wheel_joint: origin xyz=-0.02 -0.10 -0.06 -> xyz=0 -0.2 -0.25

Commit message: update

File: install/yzbot_description/share/yzbot_description/urdf/yzbot_base.urdf (robot description, URDF)
Before this commit: robot yzbot, 9 links, 8 joints
Links:
- removed link caster_back_link
- removed link caster_front_link
Joints:
- removed joint caster_back_joint
- removed joint caster_front_joint
